File: v2/roboskin_distance_IMU_WIFI.brd (EAGLE design)
At the start: 43.2 x 33 mm, 40 parts, among them IC1 CP2104, Q1 mmbt2222, Q2 mmbt2222, SW2 KMR2, U2 AP2112-3.3, U3 MCP73831T-2ACI/OT, U4 LSM6DS3DOT_INDICATION, U5 VL53L1XSMD, X1 JSTPH, X2 ESP-12, X4 20329

Commit message: adding BOM and Gerber files
Parts:
- added U$6: (no value), HIRO_graphics#PNG (6):HIRO_GRAPHICS#PNG
- moved R6 46.4 mm to (15.6, 10.6)
- moved D4 46.1 mm to (1.49, 29.3)
- moved D2 46.0 mm to (23.0, 30.1)
- moved C1 46.0 mm to (16.3, 5.08)
- moved C2 46.0 mm to (12.7, 24.1)
- moved C3 46.0 mm to (1.52, 23.6)
- moved C4 46.0 mm to (32.8, 2.79)
- moved C5 46.0 mm to (35.6, 3.68)
- moved C6 46.0 mm to (16.8, 30.5)
- moved C7 46.0 mm to (6.46, 13.9)
- moved C8 46.0 mm to (10.2, 24.1)
- moved CHG 46.0 mm to (10.5, 10.9)
- moved D1 46.0 mm to (32.8, 30.1)
- moved D3 46.0 mm to (27.9, 30.0)
- moved IC1 46.0 mm to (10.4, 15.6)
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Routing:
- net VBAT: track 33.0 -> 32.3 mm
- net GPIO15: track 6.42 -> 7.03 mm
