File: v2/roboskin_distance_IMU_WIFI.sch (EAGLE design)
At the start: 40 parts, among them IC1 CP2104, Q1 mmbt2222, Q2 mmbt2222, SW2 KMR2, U2 AP2112-3.3, U3 MCP73831T-2ACI/OT, U4 LSM6DS3DOT_INDICATION, U5 VL53L1XSMD, X1 JSTPH, X2 ESP-12, X4 20329

Commit message: adding BOM and Gerber files
Changed lines of the file:
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@@
 <part name="X2" library="microbuilder" deviceset="ESP-12S" device="" value="ESP-12"/>
 <part name="U$2" library="microbuilder" deviceset="3.3V" device=""/>
-<part name="GND3" library="supply1" deviceset="GND" device=""/>
+<part name="GND3" library="supply1" library_urn="urn:adsk.eagle:library:371" deviceset="GND" device=""/>
 <part name="R1" library="microbuilder" deviceset="RESISTOR" device="_0603_NOOUT" value="10K"/>
 <part name="U$4" library="microbuilder" deviceset="3.3V" device=""/>
@@
 <part name="U$5" library="microbuilder" deviceset="3.3V" device=""/>
 <part name="R6" library="microbuilder" deviceset="RESISTOR" device="_0603_NOOUT" value="4.7K"/>
-<part name="GND2" library="supply1" deviceset="GND" device=""/>
+<part name="GND2" library="supply1" library_urn="urn:adsk.eagle:library:371" deviceset="GND" device=""/>
 <part name="R9" library="microbuilder" deviceset="RESISTOR" device="_0603_NOOUT" value="10K"/>
 <part name="U$8" library="microbuilder" deviceset="3.3V" device=""/>
 <part name="SW2" library="microbuilder" deviceset="SWITCH_TACT_SMT" device="4.6X2.8" value="KMR2"/>
-<part name="GND6" library="supply1" deviceset="GND" device=""/>
+<part name="GND6" library="supply1" library_urn="urn:adsk.eagle:library:371" deviceset="GND" device=""/>
 <part name="D3" library="microbuilder" deviceset="LED" device="0805_NOOUTLINE" value="RED"/>
 <part name="U$14" library="microbuilder" deviceset="3.3V" device=""/>
@@
 <part name="R7" library="microbuilder" deviceset="RESISTOR" device="_0603_NOOUT" value="10K"/>
 <part name="R11" library="microbuilder" deviceset="RESISTOR" device="_0603MP" value="1K"/>
-<part name="GND1" library="supply1" deviceset="GND" device=""/>
+<part name="GND1" library="supply1" library_urn="urn:adsk.eagle:library:371" deviceset="GND" device=""/>
 <part name="U$24" library="microbuilder" deviceset="3.3V" device=""/>
 <part name="D1" library="microbuilder" deviceset="LED" device="0805_NOOUTLINE" value="RED"/>
@@
 <sheet>
 <plain>
-<text x="43.18" y="170.18" size="1.778" layer="94">POWER AND FILTERING</text>
+<text x="7.62" y="175.26" size="1.778" layer="94">POWER AND FILTERING</text>
 <wire x1="0" y1="121.92" x2="111.76" y2="121.92" width="0.1524" layer="94" style="shortdash"/>
 <wire x1="111.76" y1="121.92" x2="111.76" y2="180.34" width="0.1524" layer="94" style="shortdash"/>
