File: V2/Eagle_Files/roboskin_distance_IMU_WIFI.sch (EAGLE design)
At the start: 53 parts, among them IC1 CP2104, Q1 mmbt2222, Q2 mmbt2222, SW2 KMR2, U1 LIS3DHTR, U2 AP2112-3.3, U3 MCP, U5 VL53L1XSMD, X1 JSTPH, X2 ESP-12, X4 20329

Commit message: All versions of hardware
Parts:
- removed D5: CHG, microbuilder:LED0805_NOOUTLINE
- removed S1: (no value), SparkFun-Switches:SWITCH-SPDT-SMD-RIGHT-ANGLE
- removed TP1, TP10, TP11, TP12, TP13, TP2, TP3, TP4, TP5, TP6, TP7, TP8, TP9: TEST-POINT3X4, SparkFun-Connectors:TEST-POINT3X4
- removed X1: JSTPH, microbuilder:CON_JST_PH_2PIN
- added C4, C5: 0.1uF, SparkFun-Capacitors:0.1UF-0603-25V-(+80/-20%)
- added J1, J10, J2, J3, J4, J6, J7, J8, J9: (no value), SparkFun-Connectors:CONN_01
- added J5: (no value), SparkFun-Connectors:JST_2MM_MALE
- added Q3: ZXMP6A13FTA, SparkFun-DiscreteSemi:MOSFET-PCHANNEL
- added R17: 100k, SparkFun-Resistors:100KOHM-1/10W-1%(0603)
- added S2: POWER, SparkFun-Electromechanical:SWITCH-SPDT-SMD-A
- C2: device microbuilder:CAP_CERAMIC0805-NOOUTLINE -> SparkFun-Capacitors:10UF-0805-10V-10%
- C3, C6, C8: value 10µF -> 10uF; device microbuilder:CAP_CERAMIC0805-NOOUTLINE -> SparkFun-Capacitors:10UF-0805-10V-10%
- C7: value 1uF -> 1.0uF; device microbuilder:CAP_CERAMIC0603_NO -> SparkFun-Capacitors:1.0UF-0603-16V-10%
- D1, D2, D3: value RED -> WHITE; device microbuilder:LED0805_NOOUTLINE -> SparkFun-LED:LED-WHITE1206
- D4: value MBR120 -> WHITE; device microbuilder:DIODE-SCHOTTKYSOD-123 -> SparkFun-LED:LED-WHITE1206
- D6: value 1N4148 -> BAT20J; device microbuilder:DIODESOD-323 -> SparkFun-DiscreteSemi:DIODE-SCHOTTKY-BAT20J
- R1, R3, R4, R5, R7, R9: value 10K -> 10k; device microbuilder:RESISTOR_0603_NOOUT -> SparkFun-Resistors:10KOHM-0603-1/10W-1%
- R10, R12, R13, R2, R8: value 1K -> 1k; device microbuilder:RESISTOR_0603_NOOUT -> SparkFun-Resistors:1KOHM-0603-1/10W-1%
- R11: value 1K -> 1k; device microbuilder:RESISTOR_0603MP -> SparkFun-Resistors:1KOHM-0603-1/10W-1%
- R15, R16: value 10k -> 4.7k; device SparkFun-Resistors:10KOHM-0603-1/10W-1% -> SparkFun-Resistors:4.7KOHM-0603-1/10W-1%
- R6: value 4.7K -> 4.7k; device microbuilder:RESISTOR_0603_NOOUT -> SparkFun-Resistors:4.7KOHM-0603-1/10W-1%
- U1: value LIS3DHTR -> ISM330DLCTR; device microbuilder:ACCEL_LIS3DHTR -> ISM330:ISM330DLCTR
Connections:
- removed net N$10: D2.C, R13.2
- removed net SDO: R16.2, U1.SDO
- removed net VBAT: D4.A, S1.P
- removed net V_CHARGE: C3.1, S1.S, U3.VBAT, X1.2
- new net INMOSFET: D6.C, Q3.S, S2.S
- new net INT1: J3.1, U1.INT1
- new net INT2: J2.1, U1.INT2
- new net LIPO: C3.1, J5.+, Q3.D, U3.VBAT
- new net SDAO: J1.1, U1.SDO/SA0
- new net VDIO: C5.1, U1.VDDIO
- new net VINPUT: C6.1, R7.2, S2.P, U2.IN
- net 3.3V: now also C4.1, R15.2, R16.2; no longer R15.1, U1.ADC2, U1.VDDIO
- net ADC: now also J6.1
- net CS: now also J4.1, U1.CS; no longer D6.C
- net GND: now also C4.2, C5.2, J5.-, R17.1, U1.GND, U1.GND_2, U1.SCX, U1.SDX; no longer R16.1, U1.ADC1, U1.ADC3, U1.GND@1, U1.GND@2, U1.RES(GND), X1.1
- net GPIO13/MOSI: now also J8.1
- net GPIO14: now also J7.1
- net N$1: now also D4.C; no longer D5.C
- net N$5: now also D1.C, R13.2; no longer D3.C, R10.2
- net N$7: now also D2.C, R10.2; no longer D6.A, R15.2, U1.CS
- net N$9: now also D3.C; no longer D1.C
- net SCL: now also J9.1, R16.1
- net SDA: now also J10.1, R15.1
- net VBUS: now also D4.A, D6.A, Q3.G, R17.2; no longer C6.1, D4.C, D5.A, R7.2, U2.IN
Other:
- note added: "AUTOSWITCHING POWER"
- note added: "SPST"
- note removed: "SDO pulled low by default (R1) to set I2C address LSB to 0"
- note removed: "Set SJ1 to make I2C"
- note removed: "address LSB 1"
- moved on the sheet: C7, IC1G$1, IC1G$2, R15, R16, SW2, X4
